File: ONA_HARD/Controller.kicad_sch (KiCad schematic)
At the start: 0 parts

Commit message: chore: remove .history folders and add to gitignore
Parts:
- added 0.1µF2, 100nF3, 10μF2, 1μF2: C, Capacitor_SMD:C_0805_2012Metric, symbol Device:C
- added R16: 10k, Resistor_SMD:R_0805_2012Metric, symbol Device:R
- added R17: 10k1, Resistor_SMD:R_0805_2012Metric, symbol Device:R
- added U5: ESP32-S3-WROOM-1U, ESP32-S3-WROOM-1U:XCVR_ESP32-S3-WROOM-1U, symbol ESP32-S3-WROOM-1U:ESP32-S3-WROOM-1U
Connections:
- new net: 100nF3.1, 10μF2.1, U5.2 (3V3)
- new net 3.3v: 0.1µF2.1, 100nF3.2, 10μF2.2, 1μF2.1, R16.2, R17.1, U5.27 (IO0), U5.3 (EN)
- new net Control TDS: U5.18 (IO10)
- new net Control VFD: U5.11 (IO18)
- new net Diff Pressure Transmitter: U5.7 (IO7)
- new net Flow Sensor Pin: U5.4 (IO4)
- new net GND: 0.1µF2.2, 1μF2.2, R16.1, R17.2, U5.1 (GND), U5.40 (GND), U5.41_1 (GND), U5.41_2 (GND), U5.41_3 (GND), U5.41_4 (GND), U5.41_5 (GND), U5.41_6 (GND), U5.41_7 (GND), U5.41_8 (GND), U5.41_9 (GND)
- new net I.L.T_pin: U5.5 (IO5)
- new net Rx: U5.37 (TXD0)
- new net Rx1: U5.20 (IO12)
- new net Rx2: U5.9 (IO16)
- new net Tx: U5.36 (RXD0)
- new net Tx1: U5.19 (IO11)
- new net Tx2: U5.10 (IO17)
- new net USB D+: U5.14 (IO20)
- new net USB D-: U5.13 (IO19)
- no-connect marks 0 -> 22
