File: ONA_HARD/Power.kicad_sch (KiCad schematic)
At the start: 0 parts

Commit message: chore: remove .history folders and add to gitignore
Parts:
- added 100nF13, 22uF2: C, Capacitor_SMD:C_0805_2012Metric, symbol Device:C
- added 220uF2: C_Polarized, Capacitor_SMD:CP_Elec_6.3x7.7, symbol Device:C_Polarized
- added 33µH2: L, Inductor_SMD:L_Bourns_SRR1260, symbol Device:L
- added 470µF/50V2: C_Polarized, Capacitor_SMD:CP_Elec_10x10.5, symbol Device:C_Polarized
- added D4: SS36, Diode_SMD:D_SMC, symbol Diode:SS36
- added F2: Fuse, Fuse:Fuse_0805_2012Metric, symbol Device:Fuse
- added R28: 1Ω, Resistor_SMD:R_0805_2012Metric, symbol Device:R
- added SMBJ28A2: PTVS5V0Z1USK, Diode_SMD:D_SMB, symbol Diode:PTVS5V0Z1USK
- added SS2: D, Diode_SMD:D_SMA, symbol Device:D
- added U12: LM2596S-5, Package_TO_SOT_SMD:TO-263-5_TabPin3, symbol Regulator_Switching:LM2596S-5
- added U13: AMS1117-3.3, Package_TO_SOT_SMD:SOT-223-3_TabPin2, symbol Regulator_Linear:AMS1117-3.3
- added power2: Conn_01x02, TerminalBlock_Phoenix:TerminalBlock_Phoenix_PT-1,5-2-5.0-H_1x02_P5.00mm_Horizontal, symbol Connector_Generic:Conn_01x02
Connections:
- new net: F2.1, SS2.1 (K)
- new net: 100nF13.1, 470µF/50V2.1, F2.2, SMBJ28A2.1 (K), U12.1 (VIN)
- new net: 33µH2.1, D4.1 (K), U12.2 (OUT)
- new net +24v: SS2.2 (A), power2.2 (Pin_2)
- new net +5v: 220uF2.1, 33µH2.2, U12.4 (FB), U13.3 (VI)
- new net 24_gnd: 100nF13.2, 220uF2.2, 22uF2.2, 470µF/50V2.2, D4.2 (A), R28.2, SMBJ28A2.2 (A), U12.3 (GND), U12.5 (~{ON}/OFF), U13.1 (GND), power2.1 (Pin_1)
- new net 3.3v: 22uF2.1, R28.1, U13.2 (VO)
