File: ONA_HARD/Pressure Sensor.kicad_sch (KiCad schematic)
At the start: 0 parts

Commit message: chore: remove .history folders and add to gitignore
Parts:
- added 100nF12: C, Capacitor_SMD:C_0805_2012Metric, symbol Device:C
- added D3: BZV55B3V3, Diode_SMD:D_MiniMELF, symbol Diode:BZV55B3V3
- added I.L.T3: Conn_01x02, TerminalBlock_Phoenix:TerminalBlock_Phoenix_PT-1,5-2-5.0-H_1x02_P5.00mm_Horizontal, symbol Connector_Generic:Conn_01x02
- added R25: 1k, Resistor_SMD:R_0805_2012Metric, symbol Device:R
- added R26: 1K, Resistor_SMD:R_0805_2012Metric, symbol Device:R
- added R27: 150Ω, Resistor_SMD:R_0805_2012Metric, symbol Device:R
Connections:
- new net: I.L.T3.2 (Pin_2), R25.1, R27.2
- new net: 100nF12.1, D3.2 (A), R25.2, R26.1
- new net +24v: I.L.T3.1 (Pin_1)
- new net 24_gnd: 100nF12.2, D3.1 (K), R27.1
- new net I.L.T_pin: R26.2
