File: ONA_HARD/Prrogramming.kicad_sch (KiCad schematic)
At the start: 0 parts

Commit message: chore: remove .history folders and add to gitignore
Parts:
- added J2: USB_C_Receptacle_USB2.0_16P, Connector_USB:USB_C_Receptacle_HRO_TYPE-C-31-M-12, symbol Connector:USB_C_Receptacle_USB2.0_16P
- added R18, R19: 5.1kΩ, Resistor_SMD:R_0805_2012Metric, symbol Device:R
- added R20, R21: 22Ω, Resistor_SMD:R_0805_2012Metric, symbol Device:R
Connections:
- new net: J2.B7 (D-), R20.1
- new net: J2.A5 (CC1), R18.1
- new net: J2.A6 (D+), R21.2
- new net: J2.B5 (CC2), R19.2
- new net +5v: J2.A4 (VBUS), J2.A9 (VBUS), J2.B4 (VBUS), J2.B9 (VBUS)
- new net 3.3_gnd: J2.A1 (GND), J2.A12 (GND), J2.B1 (GND), J2.B12 (GND), R18.2, R19.1
- new net USB D+: R21.1
- new net USB D-: R20.2
- no-connect marks 0 -> 5
