File: ONA_HARD/TDS.kicad_sch (KiCad schematic)
At the start: 0 parts

Commit message: chore: remove .history folders and add to gitignore
Parts:
- added 100nF11: C, Capacitor_SMD:C_0805_2012Metric, symbol Device:C
- added R24: 120Ω, Resistor_SMD:R_0805_2012Metric, symbol Device:R
- added TDS2: Conn_01x04, TerminalBlock_Phoenix:TerminalBlock_Phoenix_PT-1,5-4-5.0-H_1x04_P5.00mm_Horizontal, symbol Connector_Generic:Conn_01x04
- added U11: MAX3485, Package_SO:SOIC-8_3.9x4.9mm_P1.27mm, symbol Interface_UART:MAX3485
Connections:
- new net: 100nF11.1, U11.8 (VCC)
- new net: R24.1, TDS2.3 (Pin_3), U11.6 (A)
- new net: R24.2, TDS2.4 (Pin_4), U11.7 (B)
- new net +24v: TDS2.1 (Pin_1)
- new net 24_gnd: TDS2.2 (Pin_2)
- new net 3.3_gnd: U11.5 (GND)
- new net 3.3v: 100nF11.2
- new net Control TDS: U11.2 (~{RE}), U11.3 (DE)
- new net Rx1: U11.1 (RO)
- new net Tx1: U11.4 (DI)
