File: ONA_HARD/STM32 & ESP32.kicad_pcb (KiCad board)
At the start: 2 copper layers, 110 x 75 mm, 86 parts, among them J1 SD Card Connector, J10 ModBus 2, J11 UART, J12 Conn_01x04_Pin, J2 24V, J3 USB_C, J4 Pressure_Sensor, J5 Flow_Sensor, J6 TDS_Sensor, J7 DIFF_Sensor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

Commit message: add docs
Connections:
- U4 pad 6: /MAX_RX -> /MAX_TX
- U4 pad 7: /MAX_TX -> /MAX_RX
Routing:
- net /MAX_TX: track 36.4 -> 41.0 mm, vias 0 -> 2
- net /MAX_RX: track 34.1 -> 32.6 mm, vias 0 -> 2
