File: ONA_HARD/STM32 & ESP32.kicad_sch (KiCad schematic)
At the start: 79 parts, among them J10 ModBus 2, J11 UART, J12 Conn_01x04_Pin, J2 24V, J3 USB_C, J4 Pressure_Sensor, J5 Flow_Sensor, J6 TDS_Sensor, J7 DIFF_Sensor, J8 TEMP_Sensor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

Commit message: add docs
Changed lines of the file:
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@@
 	)
 	(circle
-		(center 148.59 35.56)
-		(radius 0.635)
-		(stroke
-			(width 0)
-			(type default)
-			(color 132 0 132 1)
-		)
-		(fill
-			(type color)
-			(color 132 0 132 1)
-		)
-	)
-	(circle
 		(center 116.84 187.96)
 		(radius 0.635)
@@
 		)
 	)
-	(circle
-		(center 148.59 38.1)
-		(radius 0.635)
-		(stroke
-			(width 0)
-			(type default)
-			(color 132 0 132 1)
-		)
-		(fill
-			(type color)
-			(color 132 0 132 1)
-		)
-	)
 	(arc
 		(start 208.28 157.48)
@@
 	)
 	(circle
+		(center 148.59 38.1)
+		(radius 0.635)
+		(stroke
+			(width 0)
+			(type default)
+			(color 132 0 132 1)
+		)
+		(fill
+			(type color)
+			(color 132 0 132 1)
+		)
+	)
+	(circle
 		(center 203.2 48.26)
 		(radius 0.635)
@@
 	)
 	(circle
+		(center 148.59 35.56)
+		(radius 0.635)
+		(stroke
+			(width 0)
+			(type default)
+			(color 132 0 132 1)
+		)
+		(fill
+			(type color)
+			(color 132 0 132 1)
+		)
+	)
+	(circle
 		(center 203.2 43.18)
 		(radius 0.635)
@@
 		)
 	)
+	(label "MAX_RX"
+		(at 149.86 39.37 0)
+		(effects
+			(font
+				(size 1.27 1.27)
+			)
+			(justify left bottom)
+		)
+	)
 	(label "CH_TX"
 		(at 100.33 85.09 180)
@@
 		)
 	)
-	(label "MAX_TX"
-		(at 149.86 39.37 0)
-		(effects
-			(font
-				(size 1.27 1.27)
-			)
-			(justify left bottom)
-		)
-	)
 	(label "MAX_DE_RE"
 		(at 100.33 171.45 180)
@@
 		)
 	)
-	(label "MAX_RX"
-		(at 149.86 36.83 0)
-		(effects
-			(font
-				(size 1.27 1.27)
-			)
-			(justify left bottom)
-		)
-	)
 	(label "GIO0"
 		(at 152.4 189.23 180)
@@
 		)
 	)
+	(label "MAX_TX"
+		(at 149.86 36.83 0)
+		(effects
+			(font
+				(size 1.27 1.27)
+			)
+			(justify left bottom)
+		)
+	)
